File: USB-DDC.brd (EAGLE design)
At the start: 47.9 x 56.2 mm, 60 parts, among them CON1 USB, IC1 TC7WU04FU, IC2 TC7WH74FU, IC3 3.3V, IC4 3.3V, IC5 AT32UC3A3256, X1 22.5792MHz, X2 24.576MHz, X3 12MHz

Commit message: Tiny fix
Parts:
- C1, C2: value 0.1u -> 0.01u
- R1: value 10 -> 1
- X1: value 22.5792MHz -> 24.576MHz
- X2: value 24.576MHz -> 22.5792MHz
Changed lines of the file:
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@@
 </autorouter>
 <elements>
-<element name="C1" library="my_rcl" package="1608" value="0.1u" x="16.1925" y="42.8625" smashed="yes" rot="R270">
+<element name="C1" library="my_rcl" package="1608" value="0.01u" x="16.1925" y="42.8625" smashed="yes" rot="R270">
 <attribute name="NAME" x="14.2875" y="43.18" size="0.8128" layer="25" rot="R270"/>
 <attribute name="VALUE" x="14.2875" y="43.4975" size="1.27" layer="27" rot="R270"/>
@@
 <attribute name="VALUE" x="34.29" y="31.75" size="1.27" layer="28" rot="MR90"/>
 </element>
-<element name="C2" library="my_rcl" package="1608" value="0.1u" x="16.1925" y="51.1175" smashed="yes" rot="R270">
+<element name="C2" library="my_rcl" package="1608" value="0.01u" x="16.1925" y="51.1175" smashed="yes" rot="R270">
 <attribute name="NAME" x="14.605" y="51.7525" size="0.8128" layer="25" rot="R270"/>
 <attribute name="VALUE" x="14.2875" y="51.7525" size="1.27" layer="27" rot="R270"/>
@@
 <attribute name="VALUE" x="22.86" y="50.4825" size="1.27" layer="27"/>
 </element>
-<element name="R1" library="my_rcl" package="0204/7" value="10" x="6.6675" y="22.86" smashed="yes" rot="R180">
+<element name="R1" library="my_rcl" package="0204/7" value="1" x="6.6675" y="22.86" smashed="yes" rot="R180">
 <attribute name="NAME" x="6.7183" y="21.844" size="0.8128" layer="25" ratio="10" rot="R180"/>
 <attribute name="VALUE" x="5.4483" y="24.4602" size="1.27" layer="27" ratio="10" rot="R180"/>
@@
 <attribute name="VALUE" x="16.1925" y="26.035" size="1.27" layer="27"/>
 </element>
-<element name="X1" library="my_rcl" package="KC7050" value="22.5792MHz" x="21.2725" y="43.18" smashed="yes">
+<element name="X1" library="my_rcl" package="KC7050" value="24.576MHz" x="21.2725" y="43.18" smashed="yes">
 <attribute name="NAME" x="26.3525" y="41.5925" size="1.27" layer="25" font="vector" rot="R90"/>
 <attribute name="VALUE" x="17.4625" y="41.5925" size="0.8128" layer="27" font="vector" rot="R90"/>
 </element>
-<element name="X2" library="my_rcl" package="KC7050" value="24.576MHz" x="21.2725" y="51.1175" smashed="yes">
+<element name="X2" library="my_rcl" package="KC7050" value="22.5792MHz" x="21.2725" y="51.1175" smashed="yes">
 <attribute name="NAME" x="26.3525" y="49.53" size="1.27" layer="25" font="vector" rot="R90"/>
 <attribute name="VALUE" x="17.4625" y="48.895" size="0.8128" layer="27" font="vector" rot="R90"/>

Commit message: Tiny fix
Connections:
- removed net AD_LRCLK: IC5.44, IC5.90
- removed net AD_SCK: IC5.61, IC5.91
Routing:
- net AD_LRCLK: track 23.1 -> 0.00 mm
- net AD_SCK: track 18.6 -> 0.00 mm, vias 2 -> 0
- net SCK: track 57.1 -> 54.4 mm, vias 2 -> 0
Changed lines of the file:
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@@
 <?xml version="1.0" encoding="utf-8"?>
 <!DOCTYPE eagle SYSTEM "eagle.dtd">
-<eagle version="9.5.2">
+<eagle version="9.6.2">
 <drawing>
 <settings>
@@
 <setting verticaltext="up"/>
 </settings>
-<grid distance="25" unitdist="mil" unit="mil" style="lines" multiple="4" display="yes" altdistance="5" altunitdist="mil" altunit="mil"/>
+<grid distance="12.5" unitdist="mil" unit="mil" style="lines" multiple="4" display="yes" altdistance="5" altunitdist="mil" altunit="mil"/>
 <layers>
 <layer number="1" name="Top" color="4" fill="1" visible="yes" active="yes"/>
@@
 <wire x1="37.1475" y1="33.655" x2="39.37" y2="35.8775" width="0.2032" layer="1"/>
 <wire x1="37.1475" y1="33.655" x2="34.76645" y2="33.655" width="0.2032" layer="1"/>
-<wire x1="31.115" y1="21.59" x2="31.115" y2="23.1775" width="0.2032" layer="1"/>
-<wire x1="31.115" y1="23.1775" x2="30.7975" y2="23.495" width="0.2032" layer="1"/>
-<via x="30.7975" y="23.495" extent="1-16" drill="0.35"/>
-<wire x1="30.7975" y1="23.495" x2="32.7025" y2="23.495" width="0.2032" layer="16"/>
-<via x="32.7025" y="23.495" extent="1-16" drill="0.35"/>
-<wire x1="32.7025" y1="23.495" x2="32.385" y2="23.8125" width="0.2032" layer="1"/>
+<wire x1="32.385" y1="23.1775" x2="32.385" y2="20.32" width="0.2032" layer="1"/>
 <wire x1="34.1825" y1="31.0075" x2="34.1825" y2="32.19" width="0.2032" layer="1"/>
-<wire x1="32.385" y1="23.8125" x2="32.385" y2="29.21" width="0.2032" layer="1"/>
+<wire x1="32.385" y1="29.21" x2="32.385" y2="23.8125" width="0.2032" layer="1"/>
 <wire x1="32.385" y1="29.21" x2="34.1825" y2="31.0075" width="0.2032" layer="1"/>
 <wire x1="42.0325" y1="13.34" x2="40.635" y2="13.34" width="0.2032" layer="1"/>
@@
 <wire x1="40.005" y1="13.97" x2="40.005" y2="14.605" width="0.2032" layer="1"/>
 <wire x1="40.005" y1="14.605" x2="38.735" y2="15.875" width="0.2032" layer="1"/>
-<wire x1="36.83" y1="15.875" x2="31.115" y2="21.59" width="0.2032" layer="1"/>
+<wire x1="36.83" y1="15.875" x2="32.385" y2="20.32" width="0.2032" layer="1"/>
 <wire x1="38.735" y1="15.875" x2="36.83" y2="15.875" width="0.2032" layer="1"/>
 <wire x1="37.7825" y1="49.53" x2="35.2425" y2="49.53" width="0.2032" layer="1"/>
@@
 <wire x1="39.37" y1="35.8775" x2="39.37" y2="47.9425" width="0.2032" layer="1"/>
 <wire x1="39.37" y1="47.9425" x2="37.7825" y2="49.53" width="0.2032" layer="1"/>
+<wire x1="32.385" y1="23.8125" x2="32.385" y2="23.1775" width="0.2032" layer="1"/>
 </signal>
 <signal name="DATA">
@@
 <wire x1="15.1225" y1="14.54" x2="14.9225" y2="14.34" width="0.508" layer="1"/>
 </signal>
-<signal name="AD_SCK">
-<contactref element="IC5" pad="61"/>
-<contactref element="IC5" pad="91"/>
-<wire x1="31.1825" y1="32.19" x2="31.1825" y2="25.4675" width="0.2032" layer="1"/>
-<wire x1="31.1825" y1="25.4675" x2="30.7975" y2="25.0825" width="0.2032" layer="1"/>
-<via x="30.7975" y="25.0825" extent="1-16" drill="0.35"/>
-<wire x1="33.02" y1="25.0825" x2="30.7975" y2="25.0825" width="0.2032" layer="16"/>
-<via x="33.02" y="25.0825" extent="1-16" drill="0.35"/>
-<wire x1="33.02" y1="25.0825" x2="33.2625" y2="24.84" width="0.2032" layer="1"/>
-<wire x1="42.0325" y1="24.84" x2="33.2625" y2="24.84" width="0.2032" layer="1"/>
-</signal>
-<signal name="AD_LRCLK">
-<contactref element="IC5" pad="90"/>
-<contactref element="IC5" pad="44"/>
-<wire x1="31.6825" y1="32.19" x2="31.6825" y2="21.6575" width="0.2032" layer="1"/>
-<wire x1="37" y1="16.34" x2="42.0325" y2="16.34" width="0.2032" layer="1"/>
-<wire x1="31.6825" y1="21.6575" x2="37" y2="16.34" width="0.2032" layer="1"/>
-</signal>
 <signal name="N$13">
