File: USB-DDC.sch (EAGLE design)
At the start: 55 parts, among them CON1 USB, IC1 TC7WU04FU, IC2 TC7WH74FU, IC3 3.3V, IC4 3.3V, IC5 AT32UC3A3256, X1 22.5792MHz, X2 24.576MHz, X3 12MHz

Commit message: 発注
Parts:
- added DR1, DR2, DR3, DR4: HOLE-3.2, my_connector:HOLE-3.2
- added SILK1: ROBOTECHWHEELSILK-9MM, Document_Robotech:ROBOTECHWHEELSILK-9MM
- C21, C7: device my_rcl:C-1608 -> my_rcl:C-2012
- D1, D2: device my_rcl:LED-SMD2012 -> my_rcl:LED-SMD1608
- R1: device my_rcl:R-2.5 -> my_rcl:R-7.5
Connections:
- new net FREQ_VAL0: IC5G$3.PC00
- new net FREQ_VAL1: IC5G$3.PC01
- new net LED_0: IC5G$3.PX20
- new net LED_1: IC5G$3.PX46
- new net UART_RX: IC5G$2.PX04
- new net UART_TX: IC5G$2.PX05

Commit message: Tiny fix
Parts:
- C1, C2: value 0.1u -> 0.01u
- R1: value 10 -> 1
- X1: value 22.5792MHz -> 24.576MHz
- X2: value 24.576MHz -> 22.5792MHz
Changed lines of the file:
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@@
 <part name="C5" library="my_rcl" deviceset="C" device="-1608" value="0.1u"/>
 <part name="SUPPLY2" library="supply2" library_urn="urn:adsk.eagle:library:372" deviceset="GND" device=""/>
-<part name="R1" library="my_rcl" deviceset="R" device="-7.5" value="10"/>
+<part name="R1" library="my_rcl" deviceset="R" device="-7.5" value="1"/>
 <part name="FB1" library="my_rcl" deviceset="FB" device="-1608"/>
 <part name="C3" library="my_rcl" deviceset="C" device="-2012" value="10u"/>
@@
 <part name="+3V11" library="supply1" library_urn="urn:adsk.eagle:library:371" deviceset="+3V3" device=""/>
 <part name="C21" library="my_rcl" deviceset="C" device="-2012" value="10u"/>
-<part name="X1" library="my_rcl" deviceset="OSC" device="-KC7050" value="22.5792MHz"/>
-<part name="X2" library="my_rcl" deviceset="OSC" device="-KC7050" value="24.576MHz"/>
+<part name="X1" library="my_rcl" deviceset="OSC" device="-KC7050" value="24.576MHz"/>
+<part name="X2" library="my_rcl" deviceset="OSC" device="-KC7050" value="22.5792MHz"/>
 <part name="IC1" library="my_ic" deviceset="TC7WU04FU" device=""/>
 <part name="SUPPLY24" library="supply2" library_urn="urn:adsk.eagle:library:372" deviceset="GND" device=""/>
@@
 <part name="+3V12" library="supply1" library_urn="urn:adsk.eagle:library:371" deviceset="+3V3" device=""/>
 <part name="+3V13" library="supply1" library_urn="urn:adsk.eagle:library:371" deviceset="+3V3" device=""/>
-<part name="C1" library="my_rcl" deviceset="C" device="-1608" value="0.1u"/>
-<part name="C2" library="my_rcl" deviceset="C" device="-1608" value="0.1u"/>
+<part name="C1" library="my_rcl" deviceset="C" device="-1608" value="0.01u"/>
+<part name="C2" library="my_rcl" deviceset="C" device="-1608" value="0.01u"/>
 <part name="C10" library="my_rcl" deviceset="C" device="-1608" value="0.1u"/>
 <part name="C13" library="my_rcl" deviceset="C" device="-1608" value="0.1u"/>

Commit message: Tiny fix
Connections:
- removed net AD_LRCLK: IC5G$2.PX36, IC5G$3.PX26
- removed net AD_SCK: IC5G$2.PX34, IC5G$3.PX28
Changed lines of the file:
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@@
 <?xml version="1.0" encoding="utf-8"?>
 <!DOCTYPE eagle SYSTEM "eagle.dtd">
-<eagle version="9.5.2">
+<eagle version="9.6.2">
 <drawing>
 <settings>
@@
 </segment>
 </net>
-<net name="AD_SCK" class="0">
-<segment>
-<pinref part="IC5" gate="G$2" pin="PX34"/>
-<wire x1="53.34" y1="27.94" x2="48.26" y2="27.94" width="0.1524" layer="91"/>
-<label x="48.26" y="27.94" size="1.778" layer="95" rot="R180" xref="yes"/>
-</segment>
-<segment>
-<pinref part="IC5" gate="G$3" pin="PX28"/>
-<wire x1="88.9" y1="43.18" x2="83.82" y2="43.18" width="0.1524" layer="91"/>
-<label x="83.82" y="43.18" size="1.778" layer="95" rot="R180" xref="yes"/>
-</segment>
-</net>
-<net name="AD_LRCLK" class="0">
-<segment>
-<pinref part="IC5" gate="G$3" pin="PX26"/>
-<wire x1="88.9" y1="45.72" x2="83.82" y2="45.72" width="0.1524" layer="91"/>
-<label x="83.82" y="45.72" size="1.778" layer="95" rot="R180" xref="yes"/>
-</segment>
-<segment>
-<pinref part="IC5" gate="G$2" pin="PX36"/>
-<wire x1="53.34" y1="71.12" x2="48.26" y2="71.12" width="0.1524" layer="91"/>
-<label x="48.26" y="71.12" size="1.778" layer="95" rot="R180" xref="yes"/>
-</segment>
-</net>
